Commit message: started working on rrt_node

File: arm_description/urdf/arm.xacro (robot description, xacro)
@@ -3,11 +3,9 @@
 <robot name="me604" xmlns:xacro="http://www.ros.org/wiki/xacro">
   <!-- Constants for robot dimensions -->
- <xacro:property name="PI" value="3.1415926535897931"/>
-  <xacro:property name="mass" value="1" /> <!-- arbitrary value for mass -->
-  <xacro:property name="width" value="0.05" /> <!-- Square dimensions (widthxwidth) of beams -->
-  <xacro:property name="height1" value="0.1" /> <!-- Link 0 -->
-  <xacro:property name="length1" value="0.6" /> <!-- Link 2 -->
-  <xacro:property name="length2" value="0.6" /> <!-- Link 3 -->
-  <xacro:property name="camera_link" value="0.05" /> <!-- Size of square 'camera' box -->
+  <xacro:property name="mass" value="1"      /> <!-- arbitrary value for mass -->
+  <xacro:property name="width" value="0.05"  /> <!-- Square dimensions (widthxwidth) of beams -->
+  <xacro:property name="height1" value="0.5" /> <!-- Link 0 -->
+  <xacro:property name="length1" value="1" /> <!-- Link 1 -->
+  <xacro:property name="length2" value="1" /> <!-- Link 2s -->
   <xacro:include filename="$(find arm_description)/urdf/arm.gazebo" />
   <xacro:include filename="$(find arm_description)/urdf/materials.xacro" />
@@ -20,10 +18,8 @@
   </joint>
   <!-- Base Link -->
-  <xacro:link0 name="link0" height1="${height1}" width="${width}" mass="${mass/6}" />
+  <xacro:link0 name="link0" height1="${height1}" width="${width}" mass="${mass/6}"/>
   <!-- Links of the manipulator -->
   <xacro:link_arm name="link1" length="${length1}" width="${width}" mass="${mass}"/>
   <xacro:link_arm name="link2" length="${length2}" width="${width}" mass="${mass}"/>
-  <!-- laser scan link -->
-  <xacro:link0 name="hokuyo_link" height1="${height1/2}" width="${width}" mass="${mass/12}" />
   <!-- Joints of the manipulator -->
   <joint name="joint1" type="continuous">
@@ -37,13 +33,7 @@
     <parent link="link1"/>
     <child link="link2"/>
-    <origin xyz="0 ${length1 - 0.05} ${width+0.01}" rpy="0 0 0"/>
+    <origin xyz="0 ${length1 - 0.025} ${-width-0.01}" rpy="0 0 0"/>
     <axis xyz="0 0 1"/>
     <dynamics damping="0.7"/>
-  </joint>
-  <joint name="hokuyo_joint" type="fixed">
-    <axis xyz="0 0 1" />
-    <parent link="link2" />
-    <child link="hokuyo_link" />
-    <origin xyz="0 ${length2} ${width/2}" rpy="0 0 0" />
   </joint>
   <transmission name="tran1">
@@ -67,3 +57,51 @@
     </actuator>
   </transmission>
+   <joint name="hokuyo_joint" type="fixed">
+    <origin rpy="0 0 0" xyz="0.0 0.0 ${height1 + width +0.1}"/>
+    <parent link="link0"/>
+    <child link="hokuyo_link"/>
+  </joint>
+  <joint name="hokoyu_joint2" type="fixed">
+    <parent link="link1"/>
+    <child link="hokuyo_frame"/>
+    <origin xyz="0 ${length1 - 0.025} ${-2*width-0.03}" rpy="0 0 0"/>
+  </joint>
+  <link name="hokuyo_link">
+    <inertial>
+      <mass value="0.270"/>
+      <origin rpy="0 0 0" xyz="0 0 0"/>
+      <inertia ixx="2.632e-4" ixy="0" ixz="0" iyy="2.632e-4" iyz="0" izz="1.62e-4"/>
+    </inertial>
+    <visual>
+      <origin rpy="0 0 0" xyz="0 0 0"/>
+      <geometry>
+        <mesh filename="package://hector_sensors_description/meshes/hokuyo_utm30lx/hokuyo_utm_30lx.dae"/>
+      </geometry>
+    </visual>
+    <collision>
+      <origin rpy="0 0 0" xyz="0 0 -0.0115"/>
+      <geometry>
+        <box size="0.058 0.058 0.087"/>
+      </geometry>
+    </collision>
+  </link>
+  <link name="hokuyo_frame">
+    <inertial>
+      <mass value="0.270"/>
+      <origin rpy="0 0 0" xyz="0 0 0"/>
+      <inertia ixx="2.632e-4" ixy="0" ixz="0" iyy="2.632e-4" iyz="0" izz="1.62e-4"/>
+    </inertial>
+    <visual>
+      <origin rpy="0 0 0" xyz="0 0 0"/>
+      <geometry>
+        <mesh filename="package://hector_sensors_description/meshes/hokuyo_utm30lx/hokuyo_utm_30lx.dae"/>
+      </geometry>
+    </visual>
+    <collision>
+      <origin rpy="0 0 0" xyz="0 0 -0.0115"/>
+      <geometry>
+        <box size="0.058 0.058 0.087"/>
+      </geometry>
+    </collision>
+  </link>
 </robot>

Commit message: working rrt with the graphs

File: arm_description/urdf/arm.xacro (robot description, xacro)
@@ -62,9 +62,4 @@
     <child link="hokuyo_link"/>
   </joint>
-  <joint name="hokoyu_joint2" type="fixed">
-    <parent link="link1"/>
-    <child link="hokuyo_frame"/>
-    <origin xyz="0 ${length1 - 0.025} ${-2*width-0.03}" rpy="0 0 0"/>
-  </joint>
   <link name="hokuyo_link">
     <inertial>
@@ -86,22 +81,3 @@
     </collision>
   </link>
-  <link name="hokuyo_frame">
-    <inertial>
-      <mass value="0.270"/>
-      <origin rpy="0 0 0" xyz="0 0 0"/>
-      <inertia ixx="2.632e-4" ixy="0" ixz="0" iyy="2.632e-4" iyz="0" izz="1.62e-4"/>
-    </inertial>
-    <visual>
-      <origin rpy="0 0 0" xyz="0 0 0"/>
-      <geometry>
-        <mesh filename="package://hector_sensors_description/meshes/hokuyo_utm30lx/hokuyo_utm_30lx.dae"/>
-      </geometry>
-    </visual>
-    <collision>
-      <origin rpy="0 0 0" xyz="0 0 -0.0115"/>
-      <geometry>
-        <box size="0.058 0.058 0.087"/>
-      </geometry>
-    </collision>
-  </link>
 </robot>

File: arm_description/urdf/arm_description.urdf (robot description, URDF)
Before this commit: robot me604, 4 links, 3 joints
Links:
- removed link arm_base
- added link hokuyo_link, mass 0.270; collision box size=0.058 0.058 0.087; visual mesh filename=package://hector_sensors_description/meshes/hokuyo_utm30lx/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
- added link link0, mass 0.166666666667; collision box size=0.05 0.05 0.5; visual box size=0.05 0.05 0.5
- link link1: mass None -> 1; geometry collision box size=0.05 1 0.05; visual box size=0.05 1 0.05
- link link2: mass None -> 1; geometry collision box size=0.05 1 0.05; visual box size=0.05 1 0.05
Joints:
- removed joint joint_1
- removed joint joint_2
- added joint hokuyo_joint: type fixed, parent link0, child hokuyo_link, origin xyz=0.0 0.0 0.65 rpy=0 0 0
- added joint joint1: type continuous, parent link0, child link1, origin xyz=0 0 0.53 rpy=0 0 0, axis 0 0 1
- added joint joint2: type continuous, parent link1, child link2, origin xyz=0 0.975 -0.06 rpy=0 0 0, axis 0 0 1
- joint fixed: child arm_base -> link0; origin xyz=0 0 0.1 rpy=0 0 0 -> (none)
